File: genevamini.kicad_pcb (KiCad board)
At the start: 2 copper layers, 91.1 x 76.5 mm, 11 parts, among them J1 Conn_01x02

Commit message: Removed old gerbers; removed soldermask from parts of minigeneva
Routing:
- net 0V: track 12.1 -> 13.0 mm, vias 0 -> 1
- net redwheel: track 4.36 -> 4.86 mm, vias 0 -> 1
- net Net-(JP1-Pad1): track 13.0 -> 13.2 mm, vias 0 -> 1
- net redrail: vias 0 -> 1
Changed lines of the file:
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@@
-(kicad_pcb (version 20171130) (host pcbnew "(5.1.5)-3")
+(kicad_pcb (version 20171130) (host pcbnew 5.1.5-52549c5~84~ubuntu18.04.1)
   (general
     (thickness 1.6)
-    (drawings 50)
-    (tracks 14)
+    (drawings 54)
+    (tracks 21)
     (zones 0)
     (modules 11)
@@
     (mod_text_size 1 1)
     (mod_text_width 0.15)
-    (pad_size 1.4 1.4)
-    (pad_drill 0.7)
+    (pad_size 5 5)
+    (pad_drill 3.2)
     (pad_to_mask_clearance 0.051)
     (solder_mask_min_width 0.25)
@@
     (add_net redwheel)
   )
+  (module geneva:railcenter (layer F.Cu)
+    (at 100 150)
+    (fp_text reference REF** (at 0 0.5) (layer F.SilkS) hide
+      (effects (font (size 1 1) (thickness 0.15)))
+    )
+    (fp_text value railcenter (at 0 -0.5) (layer F.Fab)
+      (effects (font (size 1 1) (thickness 0.15)))
+    )
+    (pad 1 thru_hole circle (at 0 0) (size 5 5) (drill 3.2) (layers *.Cu *.Mask)
+      (net 1 5V))
+  )
+  (module geneva:jumper (layer F.Cu)
+    (at 86.66667 150)
+    (fp_text reference JP1 (at 0 2) (layer F.SilkS) hide
+      (effects (font (size 1 1) (thickness 0.15)))
+    )
+    (fp_text value Jumper_NO_Small (at 0 -2) (layer F.Fab)
+      (effects (font (size 1 1) (thickness 0.15)))
+    )
+    (pad 2 smd roundrect (at 0.4 0) (size 0.6 1) (layers F.Cu F.Mask) (roundrect_rratio 0.25)
+      (net 2 0V))
+    (pad 1 smd roundrect (at -0.4 0) (size 0.6 1) (layers F.Cu F.Mask) (roundrect_rratio 0.25)
+      (net 3 "Net-(JP1-Pad1)"))
+  )
   (module LED_THT:LED_D3.0mm (layer F.Cu)
     (at 100 91)
@@
       (net 6 5Vwheel))
     (model ${KISYS3DMOD}/LED_THT.3dshapes/LED_D3.0mm.wrl
-      (at (xyz 0 0 0))
+      (offset (xyz -1.2 0 0))
       (scale (xyz 1 1 1))
       (rotate (xyz 0 0 0))
@@
       (rotate (xyz 0 0 0))
     )
-  )
-  (module geneva:jumper (layer F.Cu)
-    (at 86.66667 150)
-    (fp_text reference JP1 (at 0 2) (layer F.SilkS) hide
-      (effects (font (size 1 1) (thickness 0.15)))
-    )
-    (fp_text value Jumper_NO_Small (at 0 -2) (layer F.Fab)
-      (effects (font (size 1 1) (thickness 0.15)))
-    )
-    (fp_circle (center 0 0) (end 0.5 0) (layer F.SilkS) (width 0.1524))
-    (pad 2 smd roundrect (at 0.4 0) (size 0.6 1) (layers F.Cu F.Mask) (roundrect_rratio 0.25)
-      (net 2 0V))
-    (pad 1 smd roundrect (at -0.4 0) (size 0.6 1) (layers F.Cu F.Mask) (roundrect_rratio 0.25)
-      (net 3 "Net-(JP1-Pad1)"))
   )
   (module Resistor_THT:R_Axial_DIN0204_L3.6mm_D1.6mm_P7.62mm_Horizontal (layer F.Cu)
@@
   )
   (module geneva:railcenter (layer F.Cu)
-    (at 100 150)
-    (fp_text reference REF** (at 0 0.5) (layer F.SilkS) hide
-      (effects (font (size 1 1) (thickness 0.15)))
-    )
-    (fp_text value railcenter (at 0 -0.5) (layer F.Fab)
-      (effects (font (size 1 1) (thickness 0.15)))
-    )
-    (pad 1 thru_hole circle (at 0 0) (size 5 5) (drill 3.2) (layers *.Cu *.Mask)
-      (net 1 5V))
-  )
-  (module geneva:railcenter (layer F.Cu)
     (at 82 150)
     (fp_text reference REF** (at 0 0.5) (layer F.SilkS) hide
@@
     (pad 1 thru_hole circle (at 0 0) (size 5 5) (drill 3) (layers *.Cu *.Mask))
   )
+  (gr_circle (center 100 100) (end 105.25 100) (layer B.Mask) (width 10.5))
+  (gr_circle (center 82 100) (end 85.5 100) (layer B.Mask) (width 7))
+  (gr_circle (center 82 150) (end 85.5 150) (layer F.Mask) (width 7.6))
+  (gr_circle (center 100 150) (end 105.25 150) (layer F.Mask) (width 11.1))
   (gr_arc (start 141 115.588457) (end 146.069004 115.108682) (angle -108.9) (layer Edge.Cuts) (width 0.15))
   (gr_line (start 138.904153 110.948154) (end 137.376606 109.135641) (layer Edge.Cuts) (width 0.05))
@@
   (segment (start 83.27 159.5) (end 90.5 159.5) (width 0.25) (layer B.Cu) (net 1))
   (segment (start 90.5 159.5) (end 100 150) (width 0.25) (layer B.Cu) (net 1))
-  (segment (start 80.73 159.5) (end 80.73 158.27) (width 0.25) (layer F.Cu) (net 2))
-  (segment (start 80.73 158.27) (end 87.06667 151.93333) (width 0.25) (layer F.Cu) (net 2))
-  (segment (start 87.06667 151.93333) (end 87.06667 150) (width 0.25) (layer F.Cu) (net 2))
-  (segment (start 86.26667 150) (end 86.26667 148.26667) (width 0.25) (layer F.Cu) (net 3))
-  (segment (start 86.26667 148.26667) (end 79 141) (width 0.25) (layer F.Cu) (net 3))
-  (segment (start 79 141) (end 78 141) (width 0.25) (layer F.Cu) (net 3))
-  (segment (start 95.66667 141) (end 100 145.33333) (width 0.25) (layer F.Cu) (net 4))
-  (segment (start 85.62 141) (end 95.66667 141) (width 0.25) (layer F.Cu) (net 4))
-  (segment (start 98.73 91.5) (end 98.73 94.06333) (width 0.25) (layer B.Cu) (net 5))
-  (segment (start 98.73 94.06333) (end 100 95.33333) (width 0.25) (layer B.Cu) (net 5))
+  (segment (start 87.06667 150) (end 87.5 150) (width 0.25) (layer F.Cu) (net 2))
+  (segment (start 87.06667 150) (end 87.399992 150) (width 0.25) (layer F.Cu) (net 2))
+  (segment (start 87.399992 150) (end 87.4 150.000008) (width 0.25) (layer F.Cu) (net 2))
+  (via (at 87.4 150.000008) (size 0.8) (drill 0.4) (layers F.Cu B.Cu) (net 2))
+  (segment (start 87.4 151.3) (end 87.4 150.000008) (width 0.25) (layer B.Cu) (net 2))
+  (segment (start 80.73 159.5) (end 80.73 157.97) (width 0.25) (layer B.Cu) (net 2))
+  (segment (start 80.73 157.97) (end 87.4 151.3) (width 0.25) (layer B.Cu) (net 2))
+  (segment (start 78 141) (end 79.5 141) (width 0.25) (layer B.Cu) (net 3))
+  (via (at 86 150) (size 0.8) (drill 0.4) (layers F.Cu B.Cu) (net 3))
+  (segment (start 79.5 141) (end 86 147.5) (width 0.25) (layer B.Cu) (net 3))
+  (segment (start 86 147.5) (end 86 150) (width 0.25) (layer B.Cu) (net 3))
+  (via (at 100 145.33333) (size 0.8) (drill 0.4) (layers F.Cu B.Cu) (net 4))
+  (segment (start 85.62 141) (end 95.66667 141) (width 0.25) (layer B.Cu) (net 4))
+  (segment (start 95.66667 141) (end 100 145.33333) (width 0.25) (layer B.Cu) (net 4))
+  (via (at 100 95.33333) (size 0.8) (drill 0.4) (layers F.Cu B.Cu) (net 5))
+  (segment (start 98.73 91) (end 98.73 94.06333) (width 0.25) (layer F.Cu) (net 5))
+  (segment (start 98.73 94.06333) (end 100 95.33333) (width 0.25) (layer F.Cu) (net 5))
   (segment (start 101.27 98.73) (end 100 100) (width 0.25) (layer F.Cu) (net 6))
   (segment (start 101.27 91.5) (end 101.27 98.73) (width 0.25) (layer F.Cu) (net 6))

Commit message: Various changes to mini version, going to order it with 2oz copper
Parts:
- moved J1 21.3 mm to (62.0, 159.0), turned to 180 degrees
- moved R1 17.7 mm to (62.0, 148.5), turned to 90 degrees
Routing:
- net redrail: track 16.2 -> 39.8 mm
- net 5V: track 20.7 -> 41.7 mm
- net 0V: track 13.0 -> 28.8 mm
- net Net-(JP1-Pad1): track 13.2 -> 28.2 mm
Other:
- board size 91.1 x 76.5 mm -> 105.1 x 76.5 mm
Changed lines of the file:
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@@
     (thickness 1.6)
     (drawings 54)
-    (tracks 21)
+    (tracks 22)
     (zones 0)
     (modules 11)
@@
     (36 B.SilkS user)
     (37 F.SilkS user)
-    (38 B.Mask user)
-    (39 F.Mask user)
+    (38 B.Mask user hide)
+    (39 F.Mask user hide)
     (40 Dwgs.User user)
     (41 Cmts.User user)
@@
     (mod_text_size 1 1)
     (mod_text_width 0.15)
-    (pad_size 5 5)
-    (pad_drill 3.2)
+    (pad_size 1.8 4.8)
+    (pad_drill 0)
     (pad_to_mask_clearance 0.051)
     (solder_mask_min_width 0.25)
@@
     (fp_line (start 2.43 2.25) (end 2.43 -2.25) (layer F.CrtYd) (width 0.05))
     (fp_line (start 2.43 -2.25) (end -2.42 -2.25) (layer F.CrtYd) (width 0.05))
-    (pad 1 thru_hole rect (at -1.27 0) (size 1.8 1.8) (drill 0.9) (layers *.Cu *.Mask)
+    (pad 1 smd rect (at -1.27 1.5) (size 1.8 4.8) (layers F.Cu F.Paste F.Mask)
       (net 5 redwheel))
-    (pad 2 thru_hole circle (at 1.27 0) (size 1.8 1.8) (drill 0.9) (layers *.Cu *.Mask)
+    (pad 2 smd rect (at 1.27 1.5) (size 1.8 4.8) (layers F.Cu F.Paste F.Mask)
       (net 6 5Vwheel))
     (model ${KISYS3DMOD}/LED_THT.3dshapes/LED_D3.0mm.wrl
@@
   )
   (module Connector_PinSocket_2.54mm:PinSocket_1x02_P2.54mm_Vertical (layer F.Cu)
-    (at 83.27 159.5 270)
+    (at 62 159 180)
     (descr "Through hole straight socket strip, 1x02, 2.54mm pitch, single row (from Kicad 4.0.7), script generated")
     (tags "Through hole socket strip THT 1x02 2.54mm single row")
-    (fp_text reference J1 (at 0 7.62 90) (layer F.SilkS) hide
-      (effects (font (size 1 1) (thickness 0.15)))
-    )
-    (fp_text value Conn_01x02 (at 0 -9.398 90) (layer F.Fab)
-      (effects (font (size 1 1) (thickness 0.15)))
-    )
-    (fp_text user %R (at 0 0 90) (layer F.Fab)
+    (fp_text reference J1 (at 0 7.62) (layer F.SilkS) hide
+      (effects (font (size 1 1) (thickness 0.15)))
+    )
+    (fp_text value Conn_01x02 (at 0 -9.398) (layer F.Fab)
+      (effects (font (size 1 1) (thickness 0.15)))
+    )
+    (fp_text user %R (at 0 0) (layer F.Fab)
       (effects (font (size 1 1) (thickness 0.15)))
     )
@@
     (fp_line (start 0.635 -1.27) (end 1.27 -0.635) (layer F.Fab) (width 0.1))
     (fp_line (start -1.27 -1.27) (end 0.635 -1.27) (layer F.Fab) (width 0.1))
-    (pad 2 thru_hole oval (at 0 2.54 270) (size 1.7 1.7) (drill 1) (layers *.Cu *.Mask)
+    (pad 2 thru_hole oval (at 0 2.54 180) (size 1.7 1.7) (drill 1) (layers *.Cu *.Mask)
       (net 2 0V))
-    (pad 1 thru_hole rect (at 0 0 270) (size 1.7 1.7) (drill 1) (layers *.Cu *.Mask)
+    (pad 1 thru_hole rect (at 0 0 180) (size 1.7 1.7) (drill 1) (layers *.Cu *.Mask)
       (net 1 5V))
     (model ${KISYS3DMOD}/Connector_PinSocket_2.54mm.3dshapes/PinSocket_1x02_P2.54mm_Vertical.wrl
@@
   )
   (module Resistor_THT:R_Axial_DIN0204_L3.6mm_D1.6mm_P7.62mm_Horizontal (layer F.Cu)
-    (at 78 141)
+    (at 62 148.5 90)
     (descr "Resistor, Axial_DIN0204 series, Axial, Horizontal, pin pitch=7.62mm, 0.167W, length*diameter=3.6*1.6mm^2, http://cdn-reichelt.de/documents/datenblatt/B400/1_4W%23YAG.pdf")
     (tags "Resistor Axial_DIN0204 series Axial Horizontal pin pitch 7.62mm 0.167W length 3.6mm diameter 1.6mm")
-    (fp_text reference R1 (at 4 0) (layer F.SilkS)
-      (effects (font (size 1 1) (thickness 0.15)))
-    )
-    (fp_text value R (at 3.81 1.92) (layer F.Fab)
+    (fp_text reference R1 (at 4 0 90) (layer F.SilkS)
+      (effects (font (size 1 1) (thickness 0.15)))
+    )
+    (fp_text value R (at 3.81 1.92 90) (layer F.Fab)
       (effects (font (size 1 1) (thickness 0.15)))
     )
@@
     (fp_line (start 2.01 0.8) (end 5.61 0.8) (layer F.Fab) (width 0.1))
     (fp_line (start 2.01 -0.8) (end 2.01 0.8) (layer F.Fab) (width 0.1))
-    (pad 2 thru_hole oval (at 7.62 0) (size 1.4 1.4) (drill 0.7) (layers *.Cu *.Mask)
+    (pad 2 thru_hole oval (at 7.62 0 90) (size 1.4 1.4) (drill 0.7) (layers *.Cu *.Mask)
       (net 4 redrail))
-    (pad 1 thru_hole circle (at 0 0) (size 1.4 1.4) (drill 0.7) (layers *.Cu *.Mask)
+    (pad 1 thru_hole circle (at 0 0 90) (size 1.4 1.4) (drill 0.7) (layers *.Cu *.Mask)
       (net 3 "Net-(JP1-Pad1)"))
     (model ${KISYS3DMOD}/Resistor_THT.3dshapes/R_Axial_DIN0204_L3.6mm_D1.6mm_P7.62mm_Horizontal.wrl
@@
     (pad 1 thru_hole circle (at 0 0) (size 5 5) (drill 3) (layers *.Cu *.Mask))
   )
+  (gr_arc (start 93.000001 149.999999) (end 104 160.999998) (angle -90) (layer Edge.Cuts) (width 0.05))
   (gr_circle (center 100 100) (end 105.25 100) (layer B.Mask) (width 10.5))
   (gr_circle (center 82 100) (end 85.5 100) (layer B.Mask) (width 7))
@@
   (gr_arc (start 150 109) (end 151.6 109) (angle -180) (layer Edge.Cuts) (width 0.15))
   (gr_line (start 148.4 91) (end 148.4 84.5) (layer Edge.Cuts) (width 0.15))
-  (gr_line (start 110 161) (end 74 161) (layer Edge.Cuts) (width 0.05))
-  (gr_line (start 74 161) (end 74 139) (layer Edge.Cuts) (width 0.05))
+  (gr_line (start 104 161) (end 60 161) (layer Edge.Cuts) (width 0.05))
+  (gr_line (start 60 161) (end 60 139) (layer Edge.Cuts) (width 0.05))
   (gr_circle (center 100 150) (end 110.5 150) (layer Dwgs.User) (width 0.15))
-  (gr_line (start 74 139) (end 110 139) (layer Edge.Cuts) (width 0.05))
+  (gr_line (start 60 139) (end 104 139) (layer Edge.Cuts) (width 0.05))
   (gr_circle (center 82 150) (end 89 150) (layer Dwgs.User) (width 0.15))
-  (gr_line (start 110 139) (end 110 161) (layer Edge.Cuts) (width 0.05))
   (gr_arc (start 82 100) (end 79.666665 104.041455) (angle -60) (layer B.Mask) (width 1))
   (gr_arc (start 82 100) (end 79.666665 95.958545) (angle -60) (layer B.Mask) (width 1))
@@
   (gr_arc (start 82 100) (end 79.666665 95.958545) (angle -60) (layer B.Cu) (width 1))
   (gr_arc (start 82 100) (end 79.666665 104.041455) (angle -60) (layer B.Cu) (width 1))
-  (segment (start 83.27 159.5) (end 90.5 159.5) (width 0.25) (layer B.Cu) (net 1))
-  (segment (start 90.5 159.5) (end 100 150) (width 0.25) (layer B.Cu) (net 1))
+  (segment (start 91 159) (end 100 150) (width 0.25) (layer B.Cu) (net 1))
+  (segment (start 62 159) (end 91 159) (width 0.25) (layer B.Cu) (net 1))
   (segment (start 87.06667 150) (end 87.5 150) (width 0.25) (layer F.Cu) (net 2))
   (segment (start 87.06667 150) (end 87.399992 150) (width 0.25) (layer F.Cu) (net 2))
   (segment (start 87.399992 150) (end 87.4 150.000008) (width 0.25) (layer F.Cu) (net 2))
   (via (at 87.4 150.000008) (size 0.8) (drill 0.4) (layers F.Cu B.Cu) (net 2))
-  (segment (start 87.4 151.3) (end 87.4 150.000008) (width 0.25) (layer B.Cu) (net 2))
-  (segment (start 80.73 159.5) (end 80.73 157.97) (width 0.25) (layer B.Cu) (net 2))
-  (segment (start 80.73 157.97) (end 87.4 151.3) (width 0.25) (layer B.Cu) (net 2))
-  (segment (start 78 141) (end 79.5 141) (width 0.25) (layer B.Cu) (net 3))
+  (segment (start 80.940008 156.46) (end 87.4 150.000008) (width 0.25) (layer B.Cu) (net 2))
+  (segment (start 62 156.46) (end 80.940008 156.46) (width 0.25) (layer B.Cu) (net 2))
   (via (at 86 150) (size 0.8) (drill 0.4) (layers F.Cu B.Cu) (net 3))
-  (segment (start 79.5 141) (end 86 147.5) (width 0.25) (layer B.Cu) (net 3))
-  (segment (start 86 147.5) (end 86 150) (width 0.25) (layer B.Cu) (net 3))
+  (segment (start 64.5 146) (end 62 148.5) (width 0.25) (layer B.Cu) (net 3))
+  (segment (start 84.5 146) (end 64.5 146) (width 0.25) (layer B.Cu) (net 3))
+  (segment (start 86 150) (end 86 147.5) (width 0.25) (layer B.Cu) (net 3))
+  (segment (start 86 147.5) (end 84.5 146) (width 0.25) (layer B.Cu) (net 3))
   (via (at 100 145.33333) (size 0.8) (drill 0.4) (layers F.Cu B.Cu) (net 4))
-  (segment (start 85.62 141) (end 95.66667 141) (width 0.25) (layer B.Cu) (net 4))
-  (segment (start 95.66667 141) (end 100 145.33333) (width 0.25) (layer B.Cu) (net 4))
-  (via (at 100 95.33333) (size 0.8) (drill 0.4) (layers F.Cu B.Cu) (net 5))
-  (segment (start 98.73 91) (end 98.73 94.06333) (width 0.25) (layer F.Cu) (net 5))
-  (segment (start 98.73 94.06333) (end 100 95.33333) (width 0.25) (layer F.Cu) (net 5))
+  (segment (start 95.54667 140.88) (end 62 140.88) (width 0.25) (layer B.Cu) (net 4))
+  (segment (start 100 145.33333) (end 95.54667 140.88) (width 0.25) (layer B.Cu) (net 4))
+  (segment (start 98.73 91) (end 99 91.27) (width 0.25) (layer F.Cu) (net 5))
+  (segment (start 99 91.27) (end 99 94.934315) (width 0.25) (layer F.Cu) (net 5))
+  (segment (start 99 94.934315) (end 99 95.5) (width 0.25) (layer F.Cu) (net 5))
+  (via (at 99 95.5) (size 0.8) (drill 0.4) (layers F.Cu B.Cu) (net 5))
   (segment (start 101.27 98.73) (end 100 100) (width 0.25) (layer F.Cu) (net 6))
   (segment (start 101.27 91.5) (end 101.27 98.73) (width 0.25) (layer F.Cu) (net 6))
